Commit message: adding colors to robot

File: robots/youbot/youbot_description/urdf/youbot_base/target_base.urdf.xacro (robot description, xacro)
@@ -68,5 +68,5 @@
         <origin xyz="0 0 ${visual_z_offset}" rpy="0 0 0"/>
         <geometry>
-          <mesh filename="package://youbot_description/meshes/youbot_base/base.dae"/>
+          <mesh filename="package://youbot_description/meshes/youbot_base/target.dae"/>
         </geometry>
         <material name="DarkGrey"/>
