Commit message: ros melodic support

File: robots/youbot/youbot_description/robots/youbot.urdf.xacro (robot description, xacro)
@@ -3,5 +3,5 @@
        xmlns:controller="http://playerstage.sourceforge.net/gazebo/xmlschema/#controller"
        xmlns:interface="http://playerstage.sourceforge.net/gazebo/xmlschema/#interface"
-       xmlns:xacro="http://playerstage.sourceforge.net/gazebo/xmlschema/#interface"
+       xmlns:xacro="http://www.ros.org/wiki/xacro/#interface"
        name="youbot" >
   <!-- The following xacro:included files set up definitions of parts of the robot body -->

File: robots/youbot/youbot_description/robots/youbot_base_laser.urdf.xacro (robot description, xacro)
@@ -3,5 +3,5 @@
        xmlns:controller="http://playerstage.sourceforge.net/gazebo/xmlschema/#controller"
        xmlns:interface="http://playerstage.sourceforge.net/gazebo/xmlschema/#interface"
-       xmlns:xacro="http://playerstage.sourceforge.net/gazebo/xmlschema/#interface"
+       xmlns:xacro="http://www.ros.org/wiki/xacro/#interface"
        name="youbot" >
   <xacro:property name="pi" value="0.0"/>

File: robots/youbot/youbot_description/robots/youbot_base_only.urdf.xacro (robot description, xacro)
@@ -3,5 +3,5 @@
        xmlns:controller="http://playerstage.sourceforge.net/gazebo/xmlschema/#controller"
        xmlns:interface="http://playerstage.sourceforge.net/gazebo/xmlschema/#interface"
-       xmlns:xacro="http://playerstage.sourceforge.net/gazebo/xmlschema/#interface"
+       xmlns:xacro="http://www.ros.org/wiki/xacro/#interface"
        name="youbot" >
   <!-- The following xacro:included files set up definitions of parts of the robot body -->

File: robots/youbot/youbot_description/robots/youbot_dual_arm.urdf.xacro (robot description, xacro)
@@ -3,5 +3,5 @@
        xmlns:controller="http://playerstage.sourceforge.net/gazebo/xmlschema/#controller"
        xmlns:interface="http://playerstage.sourceforge.net/gazebo/xmlschema/#interface"
-       xmlns:xacro="http://playerstage.sourceforge.net/gazebo/xmlschema/#interface"
+       xmlns:xacro="http://www.ros.org/wiki/xacro/#interface"
        name="youbot" >
   <!-- The following xacro:included files set up definitions of parts of the robot body -->

File: robots/youbot/youbot_description/robots/youbot_target.urdf.xacro (robot description, xacro)
@@ -3,5 +3,5 @@
        xmlns:controller="http://playerstage.sourceforge.net/gazebo/xmlschema/#controller"
        xmlns:interface="http://playerstage.sourceforge.net/gazebo/xmlschema/#interface"
-       xmlns:xacro="http://playerstage.sourceforge.net/gazebo/xmlschema/#interface"
+       xmlns:xacro="http://www.ros.org/wiki/xacro/#interface"
        name="youbot" >
   <!-- The following xacro:included files set up definitions of parts of the robot body -->

File: robots/youbot/youbot_description/urdf/common.xacro (robot description, xacro)
@@ -1,9 +1,9 @@
 <?xml version="1.0"?>
-<robot>
-	<property name="M_PI" value="3.1415926535897931" />
+<robot xmlns:xacro="http://www.ros.org/wiki/xacro/#interface">
+	<xacro:property name="M_PI" value="3.1415926535897931" />
 	<!-- Casters -->
-	<property name="cal_caster_fl" value="0.0" />
-	<property name="cal_caster_fr" value="0.0" />
-	<property name="cal_caster_bl" value="0.0" />
-	<property name="cal_caster_br" value="0.0" />
+	<xacro:property name="cal_caster_fl" value="0.0" />
+	<xacro:property name="cal_caster_fr" value="0.0" />
+	<xacro:property name="cal_caster_bl" value="0.0" />
+	<xacro:property name="cal_caster_br" value="0.0" />
 </robot>

File: robots/youbot/youbot_description/urdf/misc/cam3d_tower.urdf.xacro (robot description, xacro)
@@ -3,8 +3,8 @@
        xmlns:controller="http://playerstage.sourceforge.net/gazebo/xmlschema/#controller"
        xmlns:interface="http://playerstage.sourceforge.net/gazebo/xmlschema/#interface"
-       xmlns:xacro="http://ros.org/wiki/xacro">
-  <property name="cam3d_tower_height" value="0.49" />
-  <property name="cam3d_tower_width" value="0.03" />
-  <property name="cam3d_tower_depth" value="0.03" />
+       xmlns:xacro="http://www.ros.org/wiki/xacro/#interface">
+  <xacro:property name="cam3d_tower_height" value="0.49" />
+  <xacro:property name="cam3d_tower_width" value="0.03" />
+  <xacro:property name="cam3d_tower_depth" value="0.03" />
   <xacro:macro name="cam3d_tower" params="name parent *origin">
   	<link name="${name}_link">
@@ -29,5 +29,5 @@
     </link>
     <joint name="${name}_joint" type="fixed">
-      <insert_block name="origin" />
+      <xacro:insert_block name="origin" />
       <parent link="${parent}"/>
       <child link="${name}_link"/>

File: robots/youbot/youbot_description/urdf/sensors/asus_xtion_camera.gazebo.xacro (robot description, xacro)
@@ -3,5 +3,5 @@
       xmlns:controller="http://playerstage.sourceforge.net/gazebo/xmlschema/#controller"
       xmlns:interface="http://playerstage.sourceforge.net/gazebo/xmlschema/#interface"
-      xmlns:xacro="http://ros.org/wiki/xacro">
+      xmlns:xacro="http://www.ros.org/wiki/xacro/#interface">
 <xacro:macro name="asus_xtion_camera_gazebo" params="name">
   <xacro:asus_xtion_depth_camera_gazebo name="${name}" />

File: robots/youbot/youbot_description/urdf/sensors/asus_xtion_camera.urdf.xacro (robot description, xacro)
@@ -1,7 +1,7 @@
 <?xml version="1.0"?>
-<root xmlns:xacro="http://playerstage.sourceforge.net/gazebo/xmlschema/#interface">
+<root xmlns:xacro="http://www.ros.org/wiki/xacro/#interface">
   <xacro:include filename="$(find youbot_description)/urdf/sensors/asus_xtion_camera.gazebo.xacro" />
-  <property name="eye_x_offset" value="0.03" />
-  <property name="eye_y_offset" value="0.035" />
+  <xacro:property name="eye_x_offset" value="0.03" />
+  <xacro:property name="eye_y_offset" value="0.035" />
   <xacro:macro name="asus_xtion_eye" params="suffix parent *origin">
 	<link name="${parent}_${suffix}_frame">
@@ -15,5 +15,5 @@
 	  <parent link="${parent}_camera"/>
 	  <child link="${parent}_${suffix}_frame"/>
-	  <insert_block name="origin"/>
+	  <xacro:insert_block name="origin"/>
 	</joint>
   </xacro:macro>
@@ -40,5 +40,5 @@
     </link>
     <joint name="${name}_foot_joint" type="fixed">
-      <insert_block name="origin" />
+      <xacro:insert_block name="origin" />
       <parent link="${parent}"/>
       <child link="${name}_foot_link"/>

File: robots/youbot/youbot_description/urdf/sensors/hokuyo_urg04_laser.gazebo.xacro (robot description, xacro)
@@ -3,5 +3,5 @@
        xmlns:controller="http://playerstage.sourceforge.net/gazebo/xmlschema/#controller"
        xmlns:interface="http://playerstage.sourceforge.net/gazebo/xmlschema/#interface"
-       xmlns:xacro="http://ros.org/wiki/xacro">
+       xmlns:xacro="http://www.ros.org/wiki/xacro/#interface">
   <xacro:macro name="hokuyo_urg04_laser_gazebo" params="name ros_topic update_rate min_angle max_angle noise_stddev">
     <gazebo reference="${name}_link">

File: robots/youbot/youbot_description/urdf/sensors/hokuyo_urg04_laser.urdf.xacro (robot description, xacro)
@@ -3,10 +3,10 @@
        xmlns:controller="http://playerstage.sourceforge.net/gazebo/xmlschema/#controller"
        xmlns:interface="http://playerstage.sourceforge.net/gazebo/xmlschema/#interface"
-       xmlns:xacro="http://ros.org/wiki/xacro">
+       xmlns:xacro="http://www.ros.org/wiki/xacro/#interface">
   <xacro:include filename="$(find youbot_description)/urdf/sensors/hokuyo_urg04_laser.gazebo.xacro" />
   <xacro:macro name="hokuyo_urg04_laser" params="name parent *origin ros_topic update_rate min_angle max_angle noise_stddev">
     <joint name="${name}_hokuyo_urg04_laser_joint" type="fixed">
       <axis xyz="0 1 0" />
-      <insert_block name="origin" />
+      <xacro:insert_block name="origin" />
       <parent link="${parent}_link"/>
       <child link="${name}_link"/>

File: robots/youbot/youbot_description/urdf/sensors/hokuyo_urg04_laser_(perfect).urdf.xacro (robot description, xacro)
@@ -3,10 +3,10 @@
        xmlns:controller="http://playerstage.sourceforge.net/gazebo/xmlschema/#controller"
        xmlns:interface="http://playerstage.sourceforge.net/gazebo/xmlschema/#interface"
-       xmlns:xacro="http://ros.org/wiki/xacro">
+       xmlns:xacro="http://www.ros.org/wiki/xacro/#interface">
   <xacro:include filename="$(find youbot_description)/urdf/sensors/hokuyo_urg04_laser.gazebo.xacro" />
   <xacro:macro name="hokuyo_urg04_laser" params="name parent *origin ros_topic update_rate min_angle max_angle noise_stddev">
     <joint name="${name}_hokuyo_urg04_laser_joint" type="fixed">
       <axis xyz="0 1 0" />
-      <insert_block name="origin" />
+      <xacro:insert_block name="origin" />
       <parent link="${parent}_link"/>
       <child link="${name}_link"/>

File: robots/youbot/youbot_description/urdf/youbot_arm/arm.gazebo.xacro (robot description, xacro)
@@ -3,5 +3,5 @@
        xmlns:controller="http://playerstage.sourceforge.net/gazebo/xmlschema/#controller"
        xmlns:interface="http://playerstage.sourceforge.net/gazebo/xmlschema/#interface"
-       xmlns:xacro="http://ros.org/wiki/xacro">
+       xmlns:xacro="http://www.ros.org/wiki/xacro/#interface">
 	<xacro:macro name="youbot_arm_gazebo" params="name">
 		<gazebo reference="${name}_link_0">

File: robots/youbot/youbot_description/urdf/youbot_arm/arm.transmission.xacro (robot description, xacro)
@@ -3,5 +3,5 @@
        xmlns:controller="http://playerstage.sourceforge.net/gazebo/xmlschema/#controller"
        xmlns:interface="http://playerstage.sourceforge.net/gazebo/xmlschema/#interface"
-       xmlns:xacro="http://ros.org/wiki/xacro">
+       xmlns:xacro="http://www.ros.org/wiki/xacro/#interface">
 	<!-- reduction ratio doesn't affect the model-->
 	<!-- reduction ratio must not to be 0-->

File: robots/youbot/youbot_description/urdf/youbot_arm/arm.urdf.xacro (robot description, xacro)
@@ -3,5 +3,5 @@
         xmlns:controller="http://playerstage.sourceforge.net/gazebo/xmlschema/#controller"
         xmlns:interface="http://playerstage.sourceforge.net/gazebo/xmlschema/#interface"
-        xmlns:xacro="http://ros.org/wiki/xacro">
+        xmlns:xacro="http://www.ros.org/wiki/xacro/#interface">
 	<xacro:include filename="$(find youbot_description)/urdf/youbot_arm/arm.gazebo.xacro" />
 	<xacro:include filename="$(find youbot_description)/urdf/youbot_arm/arm.transmission.xacro" />
@@ -10,5 +10,5 @@
 		<!-- joint between base_link and arm_0_link -->
 		<joint name="${name}_joint_0" type="fixed" >
-			<insert_block name="origin" />
+			<xacro:insert_block name="origin" />
 			<parent link="${parent}" />
 			<child link="${name}_link_0" />

File: robots/youbot/youbot_description/urdf/youbot_arm/limits.urdf.xacro (robot description, xacro)
@@ -1,31 +1,31 @@
 <?xml version="1.0"?>
-<robot xmlns:xacro="http://ros.org/wiki/xacro">>
+<robot xmlns:xacro="http://www.ros.org/wiki/xacro/#interface">>
 	<!-- common properties -->
-	<property name="M_PI" value="3.1415926535897931" />
-        <property name="threshold" value="0.01" />
+	<xacro:property name="M_PI" value="3.1415926535897931" />
+        <xacro:property name="threshold" value="0.01" />
 	<!-- arm limits positions (deg) -->
-	<property name="joint_1_limit" value="${M_PI * (169 + 169) / 180}" />
-	<property name="joint_2_limit" value="${M_PI * (90 + 65) / 180}" />
-	<property name="joint_3_limit" value="${M_PI * (146 + 151) / 180}" />
-	<property name="joint_4_limit" value="${M_PI * (102.5 + 102.5) / 180}" />
-	<property name="joint_5_limit" value="${M_PI * (167.5 + 167.5) / 180}" />
-        <property name="joint_1_limit_soft" value="${M_PI * (169 + 169) / 180 - threshold}" />
-	<property name="joint_2_limit_soft" value="${M_PI * (90 + 65) / 180 - threshold}" />
-	<property name="joint_3_limit_soft" value="${M_PI * (146 + 151) / 180 - threshold}" />
-	<property name="joint_4_limit_soft" value="${M_PI * (102.5 + 102.5) / 180 - threshold}" />
-	<property name="joint_5_limit_soft" value="${M_PI * (167.5 + 167.5) / 180 - threshold}" />
+	<xacro:property name="joint_1_limit" value="${M_PI * (169 + 169) / 180}" />
+	<xacro:property name="joint_2_limit" value="${M_PI * (90 + 65) / 180}" />
+	<xacro:property name="joint_3_limit" value="${M_PI * (146 + 151) / 180}" />
+	<xacro:property name="joint_4_limit" value="${M_PI * (102.5 + 102.5) / 180}" />
+	<xacro:property name="joint_5_limit" value="${M_PI * (167.5 + 167.5) / 180}" />
+        <xacro:property name="joint_1_limit_soft" value="${M_PI * (169 + 169) / 180 - threshold}" />
+	<xacro:property name="joint_2_limit_soft" value="${M_PI * (90 + 65) / 180 - threshold}" />
+	<xacro:property name="joint_3_limit_soft" value="${M_PI * (146 + 151) / 180 - threshold}" />
+	<xacro:property name="joint_4_limit_soft" value="${M_PI * (102.5 + 102.5) / 180 - threshold}" />
+	<xacro:property name="joint_5_limit_soft" value="${M_PI * (167.5 + 167.5) / 180 - threshold}" />
 	<!-- dynamic properties : mass (kg) Alu data sheet -->
-	<property name="link_0_mass" value="0.845" />
-	<property name="link_1_mass" value="2.412" />
-	<property name="link_2_mass" value="1.155" />
-	<property name="link_3_mass" value="0.934" />
-	<property name="link_4_mass" value="0.877" />
-	<property name="link_5_mass" value="0.251" />
-	<!--<property name="link_0_mass" value="0.845" />
-	<property name="link_1_mass" value="0.1" />
-	<property name="link_2_mass" value="0.1" />
-	<property name="link_3_mass" value="0.1" />
-	<property name="link_4_mass" value="0.1" />
-	<property name="link_5_mass" value="0.1" />-->
+	<xacro:property name="link_0_mass" value="0.845" />
+	<xacro:property name="link_1_mass" value="2.412" />
+	<xacro:property name="link_2_mass" value="1.155" />
+	<xacro:property name="link_3_mass" value="0.934" />
+	<xacro:property name="link_4_mass" value="0.877" />
+	<xacro:property name="link_5_mass" value="0.251" />
+	<!--<xacro:property name="link_0_mass" value="0.845" />
+	<xacro:property name="link_1_mass" value="0.1" />
+	<xacro:property name="link_2_mass" value="0.1" />
+	<xacro:property name="link_3_mass" value="0.1" />
+	<xacro:property name="link_4_mass" value="0.1" />
+	<xacro:property name="link_5_mass" value="0.1" />-->
 	<!-- TODO: add inertia tensor-->
 	<xacro:macro name="default_origin">

File: robots/youbot/youbot_description/urdf/youbot_base/base.gazebo.xacro (robot description, xacro)
@@ -3,5 +3,5 @@
        xmlns:controller="http://playerstage.sourceforge.net/gazebo/xmlschema/#controller"
        xmlns:interface="http://playerstage.sourceforge.net/gazebo/xmlschema/#interface"
-       xmlns:xacro="http://ros.org/wiki/xacro">
+       xmlns:xacro="http://www.ros.org/wiki/xacro/#interface">
   <xacro:macro name="youbot_base_gazebo">
     <gazebo reference="youbot_base">

File: robots/youbot/youbot_description/urdf/youbot_base/base.transmission.xacro (robot description, xacro)
@@ -3,8 +3,8 @@
        xmlns:controller="http://playerstage.sourceforge.net/gazebo/xmlschema/#controller"
        xmlns:interface="http://playerstage.sourceforge.net/gazebo/xmlschema/#interface"
-       xmlns:xacro="http://ros.org/wiki/xacro">
-	<property name="wheel_mechanical_reduction" value="${624/35 * 80/18}" />
-	<property name="caster_mechanical_reduction" value="${624/35 * 80/18}" />
-  <property name="" value="0.360" />
+       xmlns:xacro="http://www.ros.org/wiki/xacro/#interface">
+	<xacro:property name="wheel_mechanical_reduction" value="${624/35 * 80/18}" />
+	<xacro:property name="caster_mechanical_reduction" value="${624/35 * 80/18}" />
+	<xacro:property name="something" value="0.360" />
 	<xacro:macro name="youbot_base_transmission">
 	<!-- front left wheel -->
@@ -12,9 +12,9 @@
       <type>transmission_interface/SimpleTransmission</type>
 			<actuator name="wheel_motor_fl">
-        <hardwareInterface>VelocityJointInterface</hardwareInterface>
+        <hardwareInterface>hardware_interface/VelocityJointInterface</hardwareInterface>
         <mechanicalReduction>${wheel_mechanical_reduction}</mechanicalReduction>
       </actuator>
 			<joint name="wheel_joint_fl">
-        <hardwareInterface>VelocityJointInterface</hardwareInterface>
+        <hardwareInterface>hardware_interface/VelocityJointInterface</hardwareInterface>
       </joint>
 		</transmission>
@@ -22,9 +22,9 @@
       <type>transmission_interface/SimpleTransmission</type>
    	  <actuator name="caster_motor_fl">
-        <hardwareInterface>VelocityJointInterface</hardwareInterface>
+        <hardwareInterface>hardware_interface/VelocityJointInterface</hardwareInterface>
         <mechanicalReduction>${caster_mechanical_reduction}</mechanicalReduction>
       </actuator>
       <joint name="caster_joint_fl">
-        <hardwareInterface>VelocityJointInterface</hardwareInterface>
+        <hardwareInterface>hardware_interface/VelocityJointInterface</hardwareInterface>
       </joint>
     </transmission>
@@ -33,9 +33,9 @@
       <type>transmission_interface/SimpleTransmission</type>
 		  <actuator name="wheel_motor_fr">
-        <hardwareInterface>VelocityJointInterface</hardwareInterface>
+        <hardwareInterface>hardware_interface/VelocityJointInterface</hardwareInterface>
         <mechanicalReduction>${wheel_mechanical_reduction}</mechanicalReduction>
       </actuator>
 		  <joint name="wheel_joint_fr">
-        <hardwareInterface>VelocityJointInterface</hardwareInterface>
+        <hardwareInterface>hardware_interface/VelocityJointInterface</hardwareInterface>
       </joint>
 	  </transmission>
@@ -43,9 +43,9 @@
       <type>transmission_interface/SimpleTransmission</type>
       <actuator name="caster_motor_fr" >
-        <hardwareInterface>VelocityJointInterface</hardwareInterface>
+        <hardwareInterface>hardware_interface/VelocityJointInterface</hardwareInterface>
         <mechanicalReduction>${caster_mechanical_reduction}</mechanicalReduction>
       </actuator>
       <joint name="caster_joint_fr">
-        <hardwareInterface>VelocityJointInterface</hardwareInterface>
+        <hardwareInterface>hardware_interface/VelocityJointInterface</hardwareInterface>
       </joint>
     </transmission>
@@ -54,9 +54,9 @@
       <type>transmission_interface/SimpleTransmission</type>
 	    <actuator name="wheel_motor_bl" >
-        <hardwareInterface>VelocityJointInterface</hardwareInterface>
+        <hardwareInterface>hardware_interface/VelocityJointInterface</hardwareInterface>
         <mechanicalReduction>${wheel_mechanical_reduction}</mechanicalReduction>
       </actuator>
 	    <joint name="wheel_joint_bl">
-        <hardwareInterface>VelocityJointInterface</hardwareInterface>
+        <hardwareInterface>hardware_interface/VelocityJointInterface</hardwareInterface>
       </joint>
 	  </transmission>
@@ -64,9 +64,9 @@
       <type>transmission_interface/SimpleTransmission</type>
       <actuator name="caster_motor_bl" >
-        <hardwareInterface>VelocityJointInterface</hardwareInterface>
+        <hardwareInterface>hardware_interface/VelocityJointInterface</hardwareInterface>
         <mechanicalReduction>${caster_mechanical_reduction}</mechanicalReduction>
       </actuator>
       <joint name="caster_joint_bl">
-        <hardwareInterface>VelocityJointInterface</hardwareInterface>
+        <hardwareInterface>hardware_interface/VelocityJointInterface</hardwareInterface>
       </joint>
     </transmission>
@@ -75,9 +75,9 @@
       <type>transmission_interface/SimpleTransmission</type>
 	    <actuator name="wheel_motor_br" >
-        <hardwareInterface>VelocityJointInterface</hardwareInterface>
+        <hardwareInterface>hardware_interface/VelocityJointInterface</hardwareInterface>
         <mechanicalReduction>${wheel_mechanical_reduction}</mechanicalReduction>
       </actuator>
 		  <joint name="wheel_joint_br">
-        <hardwareInterface>VelocityJointInterface</hardwareInterface>
+        <hardwareInterface>hardware_interface/VelocityJointInterface</hardwareInterface>
       </joint>
 	  </transmission>
@@ -85,9 +85,9 @@
       <type>transmission_interface/SimpleTransmission</type>
       <actuator name="caster_motor_br" >
-        <hardwareInterface>VelocityJointInterface</hardwareInterface>
+        <hardwareInterface>hardware_interface/VelocityJointInterface</hardwareInterface>
         <mechanicalReduction>${caster_mechanical_reduction}</mechanicalReduction>
       </actuator>
       <joint name="caster_joint_br">
-        <hardwareInterface>VelocityJointInterface</hardwareInterface>
+        <hardwareInterface>hardware_interface/VelocityJointInterface</hardwareInterface>
       </joint>
     </transmission>
