Commit message: ros melodic support

File: robots/youbot/youbot_description/urdf/youbot_base/base.urdf.xacro (robot description, xacro)
@@ -3,33 +3,33 @@
        xmlns:controller="http://playerstage.sourceforge.net/gazebo/xmlschema/#controller"
        xmlns:interface="http://playerstage.sourceforge.net/gazebo/xmlschema/#interface"
-       xmlns:xacro="http://ros.org/wiki/xacro">
+       xmlns:xacro="http://www.ros.org/wiki/xacro/#interface">
   <!-- sensors -->
   <xacro:include filename="$(find youbot_description)/urdf/youbot_base/base.gazebo.xacro"/>
   <xacro:include filename="$(find youbot_description)/urdf/youbot_base/base.transmission.xacro"/>
   <!-- simplified box collision geometry for base -->
-  <property name="base_size_x" value="0.570"/>
-  <property name="base_size_y" value="0.360"/>
-  <property name="base_size_z" value="0.100"/>
-  <property name="base_mass" value="22.0"/>
-  <property name="caster_offset_x" value="0.228"/>
-  <property name="caster_offset_y" value="0.158"/>
-  <property name="caster_offset_z" value="-0.034"/>
-  <property name="caster_mass" value="0.1"/>
-  <property name="wheel_offset_x" value="0.0"/>
-  <property name="wheel_offset_y" value="0.0"/>
-  <property name="wheel_offset_z" value="0.0"/>
-  <property name="wheel_mass" value="0.4"/>
-  <property name="wheel_radius" value="0.05"/>
-  <property name="wheel_length" value="0.005"/>
-  <property name="caster_joint_damping" value="1.0"/>
-  <property name="caster_joint_friction" value="1.0"/>
-  <property name="caster_joint_effort" value="30"/>
-  <property name="caster_joint_velocity" value="10"/>
-  <property name="caster_joint_safety_k_velocity" value="10.0"/>
-  <property name="wheel_joint_damping" value="1.0"/>
-  <property name="wheel_joint_friction" value="1.0"/>
-  <property name="wheel_joint_effort" value="30"/>
-  <property name="wheel_joint_velocity" value="10"/>
-  <property name="wheel_joint_safety_k_velocity" value="10.0"/>
+  <xacro:property name="base_size_x" value="0.570"/>
+  <xacro:property name="base_size_y" value="0.360"/>
+  <xacro:property name="base_size_z" value="0.100"/>
+  <xacro:property name="base_mass" value="22.0"/>
+  <xacro:property name="caster_offset_x" value="0.228"/>
+  <xacro:property name="caster_offset_y" value="0.158"/>
+  <xacro:property name="caster_offset_z" value="-0.034"/>
+  <xacro:property name="caster_mass" value="0.1"/>
+  <xacro:property name="wheel_offset_x" value="0.0"/>
+  <xacro:property name="wheel_offset_y" value="0.0"/>
+  <xacro:property name="wheel_offset_z" value="0.0"/>
+  <xacro:property name="wheel_mass" value="0.4"/>
+  <xacro:property name="wheel_radius" value="0.05"/>
+  <xacro:property name="wheel_length" value="0.005"/>
+  <xacro:property name="caster_joint_damping" value="1.0"/>
+  <xacro:property name="caster_joint_friction" value="1.0"/>
+  <xacro:property name="caster_joint_effort" value="30"/>
+  <xacro:property name="caster_joint_velocity" value="10"/>
+  <xacro:property name="caster_joint_safety_k_velocity" value="10.0"/>
+  <xacro:property name="wheel_joint_damping" value="1.0"/>
+  <xacro:property name="wheel_joint_friction" value="1.0"/>
+  <xacro:property name="wheel_joint_effort" value="30"/>
+  <xacro:property name="wheel_joint_velocity" value="10"/>
+  <xacro:property name="wheel_joint_safety_k_velocity" value="10.0"/>
   <xacro:macro name="youbot_base" params="name">
     <link name="${name}_footprint">

File: robots/youbot/youbot_description/urdf/youbot_base/target_base.urdf.xacro (robot description, xacro)
@@ -3,34 +3,34 @@
        xmlns:controller="http://playerstage.sourceforge.net/gazebo/xmlschema/#controller"
        xmlns:interface="http://playerstage.sourceforge.net/gazebo/xmlschema/#interface"
-       xmlns:xacro="http://ros.org/wiki/xacro">
+       xmlns:xacro="http://www.ros.org/wiki/xacro/#interface">
   <!-- sensors -->
   <xacro:include filename="$(find youbot_description)/urdf/youbot_base/base.gazebo.xacro"/>
   <xacro:include filename="$(find youbot_description)/urdf/youbot_base/base.transmission.xacro"/>
   <!-- simplified box collision geometry for base -->
-  <property name="base_size_x" value="0.90"/>
-  <property name="base_size_y" value="0.90"/>
-  <property name="base_size_z" value="0.5"/>
-  <property name="base_mass" value="22.0"/>
-  <property name="visual_z_offset" value="-0.16"/>
-  <property name="caster_offset_x" value="0.228"/>
-  <property name="caster_offset_y" value="0.158"/>
-  <property name="caster_offset_z" value="-0.034"/>
-  <property name="caster_mass" value="0.1"/>
-  <property name="wheel_offset_x" value="0.0"/>
-  <property name="wheel_offset_y" value="0.0"/>
-  <property name="wheel_offset_z" value="0.0"/>
-  <property name="wheel_mass" value="0.4"/>
-  <property name="wheel_radius" value="0.05"/>
-  <property name="wheel_length" value="0.005"/>
-  <property name="caster_joint_damping" value="1.0"/>
-  <property name="caster_joint_friction" value="1.0"/>
-  <property name="caster_joint_effort" value="30"/>
-  <property name="caster_joint_velocity" value="10"/>
-  <property name="caster_joint_safety_k_velocity" value="10.0"/>
-  <property name="wheel_joint_damping" value="1.0"/>
-  <property name="wheel_joint_friction" value="1.0"/>
-  <property name="wheel_joint_effort" value="30"/>
-  <property name="wheel_joint_velocity" value="10"/>
-  <property name="wheel_joint_safety_k_velocity" value="10.0"/>
+  <xacro:property name="base_size_x" value="0.90"/>
+  <xacro:property name="base_size_y" value="0.90"/>
+  <xacro:property name="base_size_z" value="0.5"/>
+  <xacro:property name="base_mass" value="22.0"/>
+  <xacro:property name="visual_z_offset" value="-0.16"/>
+  <xacro:property name="caster_offset_x" value="0.228"/>
+  <xacro:property name="caster_offset_y" value="0.158"/>
+  <xacro:property name="caster_offset_z" value="-0.034"/>
+  <xacro:property name="caster_mass" value="0.1"/>
+  <xacro:property name="wheel_offset_x" value="0.0"/>
+  <xacro:property name="wheel_offset_y" value="0.0"/>
+  <xacro:property name="wheel_offset_z" value="0.0"/>
+  <xacro:property name="wheel_mass" value="0.4"/>
+  <xacro:property name="wheel_radius" value="0.05"/>
+  <xacro:property name="wheel_length" value="0.005"/>
+  <xacro:property name="caster_joint_damping" value="1.0"/>
+  <xacro:property name="caster_joint_friction" value="1.0"/>
+  <xacro:property name="caster_joint_effort" value="30"/>
+  <xacro:property name="caster_joint_velocity" value="10"/>
+  <xacro:property name="caster_joint_safety_k_velocity" value="10.0"/>
+  <xacro:property name="wheel_joint_damping" value="1.0"/>
+  <xacro:property name="wheel_joint_friction" value="1.0"/>
+  <xacro:property name="wheel_joint_effort" value="30"/>
+  <xacro:property name="wheel_joint_velocity" value="10"/>
+  <xacro:property name="wheel_joint_safety_k_velocity" value="10.0"/>
   <xacro:macro name="youbot_base" params="name">
     <link name="${name}_footprint">
